Commit message: Changed origin to be facing the right direction

File: ros/catkin_ws/src/robots_with_aruco/urdf/tb3_3.urdf.xacro (robot description, xacro)
@@ -15,5 +15,5 @@
     <parent link="base_footprint"/>
     <child link="base_link" />
-    <origin xyz="0 0 0.010" rpy="0 0 3.14159"/>
+    <origin xyz="0 0 0.010" rpy="0 0 0"/>
   </joint>
   <link name="base_link">
