Commit message: Flipped markers 2 and 4 on each robot to fix relative position bug.

File: ros/catkin_ws/src/robots_with_aruco/urdf/tb3_1.urdf.xacro (robot description, xacro)
@@ -7,7 +7,7 @@
   <xacro:property name="cube_length" value="0.1" />
   <xacro:property name="front_tag" value="11" />
-  <xacro:property name="right_tag" value="12" />
+  <xacro:property name="right_tag" value="14" />
   <xacro:property name="back_tag" value="13" />
-  <xacro:property name="left_tag" value="14" />
+  <xacro:property name="left_tag" value="12" />
   <xacro:property name="artag_offset" value="${cube_length/2+0.001}" />
   <link name="base_footprint"/>

File: ros/catkin_ws/src/robots_with_aruco/urdf/tb3_2.urdf.xacro (robot description, xacro)
@@ -7,7 +7,7 @@
   <xacro:property name="cube_length" value="0.1" />
   <xacro:property name="front_tag" value="21" />
-  <xacro:property name="right_tag" value="22" />
+  <xacro:property name="right_tag" value="24" />
   <xacro:property name="back_tag" value="23" />
-  <xacro:property name="left_tag" value="24" />
+  <xacro:property name="left_tag" value="22" />
   <xacro:property name="artag_offset" value="${cube_length/2+0.001}" />
   <link name="base_footprint"/>

File: ros/catkin_ws/src/robots_with_aruco/urdf/tb3_3.urdf.xacro (robot description, xacro)
@@ -7,7 +7,7 @@
   <xacro:property name="cube_length" value="0.1" />
   <xacro:property name="front_tag" value="31" />
-  <xacro:property name="right_tag" value="32" />
+  <xacro:property name="right_tag" value="34" />
   <xacro:property name="back_tag" value="33" />
-  <xacro:property name="left_tag" value="34" />
+  <xacro:property name="left_tag" value="32" />
   <xacro:property name="artag_offset" value="${cube_length/2+0.001}" />
   <link name="base_footprint"/>

Commit message: Updated gitignore and fixed aruco offset to be above robot origin

File: ros/catkin_ws/src/robots_with_aruco/urdf/tb3_1.urdf.xacro (robot description, xacro)
@@ -3,5 +3,5 @@
   <xacro:include filename="$(find robots_with_aruco)/urdf/common_properties.xacro"/>
   <xacro:include filename="$(find robots_with_aruco)/urdf/turtlebot3_1.gazebo.xacro"/>
-  <xacro:property name="cube_x_offset" value="-0.1" />
+  <xacro:property name="cube_x_offset" value="0" />
   <xacro:property name="cube_z_offset" value="0.2" />
   <xacro:property name="cube_length" value="0.1" />

File: ros/catkin_ws/src/robots_with_aruco/urdf/tb3_2.urdf.xacro (robot description, xacro)
@@ -3,5 +3,5 @@
   <xacro:include filename="$(find robots_with_aruco)/urdf/common_properties.xacro"/>
   <xacro:include filename="$(find robots_with_aruco)/urdf/turtlebot3_1.gazebo.xacro"/>
-  <xacro:property name="cube_x_offset" value="-0.1" />
+  <xacro:property name="cube_x_offset" value="0" />
   <xacro:property name="cube_z_offset" value="0.2" />
   <xacro:property name="cube_length" value="0.1" />

File: ros/catkin_ws/src/robots_with_aruco/urdf/tb3_3.urdf.xacro (robot description, xacro)
@@ -3,5 +3,5 @@
   <xacro:include filename="$(find robots_with_aruco)/urdf/common_properties.xacro"/>
   <xacro:include filename="$(find robots_with_aruco)/urdf/turtlebot3_1.gazebo.xacro"/>
-  <xacro:property name="cube_x_offset" value="-0.1" />
+  <xacro:property name="cube_x_offset" value="0" />
   <xacro:property name="cube_z_offset" value="0.2" />
   <xacro:property name="cube_length" value="0.1" />
